File: hardware/Kicad/ignition-system/ignition-system.kicad_pcb (KiCad board)
At the start: 2 copper layers, 92 x 60.2 mm, 27 parts, among them J1 Screw_Terminal_01x02, SW1 SW_Push, SW2 SW_SPDT

Commit message: chore(update): bump inputs
Parts:
- SW2: footprint Connector_PinHeader_2.54mm:PinHeader_1x03_P2.54mm_Vertical -> Button_Switch_THT:SW_E-Switch_EG1224_SPDT_Angled
Connections:
- ModuloDeCarga1 pad 1: unconnected-(ModuloDeCarga1-TEMP-Pad1) -> GND
- ModuloDeCarga1 pad 8: VCC -> VBUS
- SW2 pad 1: unconnected-(SW2-A-Pad1) -> VSYS
- SW2 pad 2: VSYS -> Net-(J1-Pin_1)
- SW2 pad 3: Net-(J1-Pin_1) -> GND
